File: 4 GC port esd board (for wii mini)/4 GC port esd board (for wii mini).kicad_pcb (KiCad board)
At the start: 2 copper layers, 17.5 x 46 mm, 20 parts, among them J1 port 4, J2 port 1, J3 port 2, J4 port 3, J5 power, J6 controller ports

Commit message: added silk
Other:
- board text added: "0.1uF caps"
